File: HW2/Swissler_HW2.sch (EAGLE design)
At the start: 22 parts, among them J1 USB-MB-H

Commit message: Preliminary Board Layout
Connections:
- net N$7 renamed VCAP
Changed lines of the file:
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@@
 </segment>
 </net>
-<net name="N$7" class="0">
+<net name="VCAP" class="0">
 <segment>
 <pinref part="U$1" gate="G$1" pin="20.VCAP"/>
@@
 <pinref part="C5" gate="G$1" pin="+"/>
 <wire x1="109.22" y1="43.18" x2="109.22" y2="40.64" width="0.1524" layer="91"/>
+<label x="93.98" y="38.1" size="1.778" layer="95"/>
 </segment>
 </net>
