File: HW2/Swissler_HW2.sch (EAGLE design)
At the start: 22 parts, among them J1 USB-MB-H

Commit message: Initial Board
Connections:
- net N$1 renamed VBUS
- net N$7 renamed VCAP
- net +5V: now also U$2.1; no longer U$2.3
Changed lines of the file:
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@@
 <instance part="U$1" gate="G$1" x="60.96" y="60.96"/>
 <instance part="J1" gate="G$1" x="35.56" y="134.62" rot="R180"/>
-<instance part="U$2" gate="G$1" x="66.04" y="147.32"/>
+<instance part="U$2" gate="G$1" x="66.04" y="147.32" rot="MR0"/>
 <instance part="U$3" gate="G$1" x="132.08" y="132.08"/>
 <instance part="LED1" gate="G$1" x="180.34" y="129.54"/>
@@
 </segment>
 </net>
-<net name="N$1" class="0">
+<net name="VBUS" class="0">
 <segment>
 <pinref part="J1" gate="G$1" pin="VBUS"/>
@@
 <net name="+5V" class="0">
 <segment>
-<pinref part="U$2" gate="G$1" pin="3"/>
-<wire x1="73.66" y1="134.62" x2="73.66" y2="132.08" width="0.1524" layer="91"/>
 <pinref part="U$3" gate="G$1" pin="2.VIN"/>
-<wire x1="73.66" y1="132.08" x2="88.9" y2="132.08" width="0.1524" layer="91"/>
 <pinref part="P+1" gate="1" pin="+5V"/>
 <wire x1="88.9" y1="132.08" x2="104.14" y2="132.08" width="0.1524" layer="91"/>
 <wire x1="104.14" y1="132.08" x2="114.3" y2="132.08" width="0.1524" layer="91"/>
-<wire x1="88.9" y1="137.16" x2="88.9" y2="132.08" width="0.1524" layer="91"/>
-<junction x="88.9" y="132.08"/>
+<wire x1="88.9" y1="137.16" x2="88.9" y2="134.62" width="0.1524" layer="91"/>
 <pinref part="C3" gate="G$1" pin="1"/>
+<wire x1="88.9" y1="134.62" x2="88.9" y2="132.08" width="0.1524" layer="91"/>
 <wire x1="104.14" y1="129.54" x2="104.14" y2="132.08" width="0.1524" layer="91"/>
 <junction x="104.14" y="132.08"/>
+<pinref part="U$2" gate="G$1" pin="1"/>
+<wire x1="73.66" y1="134.62" x2="88.9" y2="134.62" width="0.1524" layer="91"/>
+<junction x="88.9" y="134.62"/>
 </segment>
 <segment>
@@
 </segment>
 </net>
-<net name="N$7" class="0">
+<net name="VCAP" class="0">
 <segment>
 <pinref part="U$1" gate="G$1" pin="20.VCAP"/>
@@
 <pinref part="C5" gate="G$1" pin="+"/>
 <wire x1="109.22" y1="43.18" x2="109.22" y2="40.64" width="0.1524" layer="91"/>
+<label x="93.98" y="38.1" size="1.778" layer="95"/>
 </segment>
 </net>
@@
 </sheet>
 </sheets>
+<errors>
+</errors>
 </schematic>
 </drawing>
