File: HW2/Swissler_HW2-3.sch (EAGLE design)
At the start: 22 parts, among them J1 USB-MB-H

Commit message: Added Silkscreen images
Parts:
- U$2: value SLIDE -> ON
Connections:
- net N$2 renamed OSC1
- net N$3 renamed OSC2
Changed lines of the file:
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@@
 <part name="U$1" library="Swissler_HW2" deviceset="PIC32MX250F128B" device=""/>
 <part name="J1" library="Swissler_HW2" deviceset="USB" device="-MB-H"/>
-<part name="U$2" library="Swissler_HW2" deviceset="SLIDE" device=""/>
+<part name="U$2" library="Swissler_HW2" deviceset="SLIDE" device="" value="ON"/>
 <part name="U$3" library="Swissler_HW2" deviceset="MMCP1702" device=""/>
 <part name="LED1" library="led" deviceset="LED" device="3MM" value="RED"/>
@@
 <instance part="U$1" gate="G$1" x="60.96" y="60.96"/>
 <instance part="J1" gate="G$1" x="35.56" y="134.62" rot="R180"/>
-<instance part="U$2" gate="G$1" x="66.04" y="147.32"/>
+<instance part="U$2" gate="G$1" x="66.04" y="147.32" rot="MR0"/>
 <instance part="U$3" gate="G$1" x="132.08" y="132.08"/>
 <instance part="LED1" gate="G$1" x="180.34" y="129.54"/>
@@
 <net name="+5V" class="0">
 <segment>
-<pinref part="U$2" gate="G$1" pin="3"/>
-<wire x1="73.66" y1="134.62" x2="73.66" y2="132.08" width="0.1524" layer="91"/>
 <pinref part="U$3" gate="G$1" pin="2.VIN"/>
-<wire x1="73.66" y1="132.08" x2="88.9" y2="132.08" width="0.1524" layer="91"/>
 <pinref part="P+1" gate="1" pin="+5V"/>
 <wire x1="88.9" y1="132.08" x2="104.14" y2="132.08" width="0.1524" layer="91"/>
 <wire x1="104.14" y1="132.08" x2="114.3" y2="132.08" width="0.1524" layer="91"/>
+<pinref part="C3" gate="G$1" pin="1"/>
 <wire x1="88.9" y1="137.16" x2="88.9" y2="132.08" width="0.1524" layer="91"/>
-<junction x="88.9" y="132.08"/>
-<pinref part="C3" gate="G$1" pin="1"/>
 <wire x1="104.14" y1="129.54" x2="104.14" y2="132.08" width="0.1524" layer="91"/>
 <junction x="104.14" y="132.08"/>
+<pinref part="U$2" gate="G$1" pin="3"/>
+<wire x1="58.42" y1="134.62" x2="58.42" y2="127" width="0.1524" layer="91"/>
+<wire x1="58.42" y1="127" x2="88.9" y2="127" width="0.1524" layer="91"/>
+<wire x1="88.9" y1="127" x2="88.9" y2="132.08" width="0.1524" layer="91"/>
+<junction x="88.9" y="132.08"/>
 </segment>
 <segment>
@@
 </segment>
 </net>
-<net name="N$2" class="0">
+<net name="OSC1" class="0">
 <segment>
 <pinref part="U$9" gate="G$1" pin="3.OSC2"/>
@@
 </segment>
 </net>
-<net name="N$3" class="0">
+<net name="OSC2" class="0">
 <segment>
 <pinref part="U$9" gate="G$1" pin="1.OSC1"/>
